Commit message: Added Contact Sensor to F1Tenth Model

File: src/simulator/racecar-simulator/racecar_description/urdf/racecar_gen.xacro (robot description, xacro)
@@ -198,4 +198,29 @@
     <child link="imu_link"/>
   </joint>
+  <!--contact sensor link-->
+  <link name="contact_link">
+  <inertial>
+    <xacro:chassis_inertial_params />
+  </inertial>
+  <visual>
+    <origin rpy="0 0 0" xyz="0 0 0"/>
+    <geometry>
+      <box size="1.0 1.0 0.01"/><!--<box size="0.001 0.001 0.001"/>-->
+    </geometry>
+  </visual>
+  <collision>
+    <origin rpy="0 0 0" xyz="0 0 0"/>
+    <geometry>
+      <box size="1.0 1.0 .01"/>
+      <material name="grey" />
+    </geometry>
+  </collision>
+</link>
+<joint name="contact_joint" type="fixed">
+    <axis xyz="0 0 1"/> <!-- 0 1 0 -->
+    <origin xyz="0.0 0 0.0"/>
+    <parent link="chassis"/>
+    <child link="contact_link"/>
+  </joint>
   <!-- zed camera -->
   <link name="zed_camera_link">

Commit message: Contact Sensor Now Works

File: src/simulator/racecar-simulator/racecar_description/urdf/racecar_gen.xacro (robot description, xacro)
@@ -198,20 +198,22 @@
     <child link="imu_link"/>
   </joint>
-  <!--contact sensor link-->
+  <!--contact sensor link
+    This thing was annoying af to put in here
+    Toggle the visual to display it
+  -->
   <link name="contact_link">
   <inertial>
     <xacro:chassis_inertial_params />
   </inertial>
-  <visual>
-    <origin rpy="0 0 0" xyz="0 0 0"/>
-    <geometry>
-      <box size="1.0 1.0 0.01"/><!--<box size="0.001 0.001 0.001"/>-->
-    </geometry>
-  </visual>
+  <!--<visual>
+    <origin rpy="0 0 0" xyz="0.18 0 0.1"/>
+    <geometry>
+      <box size="0.5 0.3 0.001"/>
+    </geometry>
+  </visual>-->
   <collision>
-    <origin rpy="0 0 0" xyz="0 0 0"/>
-    <geometry>
-      <box size="1.0 1.0 .01"/>
-      <material name="grey" />
+    <origin rpy="0 0 0" xyz="0.18 0 0.1"/>
+    <geometry>
+      <box size="0.5 0.3 0.001"/>
     </geometry>
   </collision>
